File: electronics/bldc_driver/bldc_driver.brd (EAGLE design)
At the start: 48 x 30 mm, 42 parts, among them Q1 MOSFET-N, Q2 MOSFET-N, Q3 MOSFET-N, Q4 MOSFET-N, Q5 MOSFET-N, Q6 MOSFET-N, X1 LOGIC, X3 MICROMATCH-10

Commit message: Prepared bldc driver for order
Routing:
- net GND: track 20.1 -> 22.2 mm, vias 10 -> 45
